File: device_adapters.kicad_sch (KiCad schematic)
At the start: 57 parts, among them J1 20pin, J2 VPP pulldown, J3 18LFxxJxx, U10 SPI FLASH@3.3V, U13 PIC12/16/18@3.3V 28p, U14 PIC30@5V 18/28p, U15 PIC12/16/18@3.3V 8/14/18/20p, U16 AVR Tiny x61A, U17 AVR 20/28p, U18 PIC24-33@3.3V 14/18p, U19 AVR Tiny 8p, U20 AVR Tiny 14p, U22 PIC24-33@3.3V 20/28p, U23 10F20x 8p, U3 uWire, U4 10F20x SOT-23, U6 SPI, U7 PIC12/16/18@5V 28p, U8 I2C/UNIO, U9 PIC12/16/18@5V 8/14/16/20p

Commit message: Add schematic
Other:
- title: Openprog+ -> Openprog All-In-One
Changed lines of the file:
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@@
   (paper "A3")
   (title_block
-    (title "Openprog+")
+    (title "Openprog All-In-One")
     (date "2023-09-02")
     (rev "1.0")
